File: pcb/ili9341_controller.kicad_pcb (KiCad board)
At the start: 2 copper layers, 162 parts, among them J1 USB_B_Micro, J2 RP_SWD_CONN, J3 CONN_RP2040, J4 CONN_FPGA, J5 CONN_TFT, J6 CONN_PWR, J7 PWR_JUMPERS, Q1 NPN, Q2 NPN, Q3 NPN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

Commit message: place components on pcb in groups
Parts:
- moved R19 248.7 mm to (260.9, 144.0)
- moved R21 247.3 mm to (260.9, 145.9)
- moved R22 246.9 mm to (260.9, 147.4)
- moved R23 246.7 mm to (261.0, 149.3)
- moved R24 246.3 mm to (261.0, 151.0)
- moved R20 246.2 mm to (260.9, 140.8)
- moved R25 246.1 mm to (261.0, 153.0)
- moved C15 239.5 mm to (224.3, 157.5), turned to 90 degrees
- moved C13 237.5 mm to (224.3, 149.1), turned to 90 degrees
- moved C14 235.8 mm to (218.0, 157.5), turned to 90 degrees
- moved R27 233.6 mm to (275.7, 55.5)
- moved C34 233.6 mm to (265.4, 45.6), turned to 90 degrees
- moved C35 232.0 mm to (263.9, 45.6), turned to 90 degrees
- moved Q1 230.4 mm to (268.4, 144.9)
- moved Q2 230.0 mm to (268.4, 148.4)
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Routing:
- net +3V3: track 0.00 -> 3.35 mm

Commit message: place and route out all components
Parts:
- moved Q3 232.3 mm to (42.6, 97.4), turned to -90 degrees
- moved R25 228.2 mm to (41.6, 90.0), turned to -90 degrees
- moved Q2 228.1 mm to (46.1, 97.4), turned to -90 degrees
- moved R24 225.9 mm to (43.5, 90.0), turned to -90 degrees
- moved R23 223.8 mm to (45.2, 90.0), turned to -90 degrees
- moved Q1 223.8 mm to (49.7, 97.4), turned to -90 degrees
- moved D10 223.7 mm to (43.5, 86.4), turned to 90 degrees
- moved R22 221.4 mm to (47.1, 90.0), turned to -90 degrees
- moved R21 219.3 mm to (48.7, 90.0), turned to -90 degrees
- moved D9 219.2 mm to (47.1, 86.4), turned to 90 degrees
- moved R19 217.0 mm to (50.6, 90.0), turned to -90 degrees
- moved D7 214.7 mm to (50.6, 86.4), turned to 90 degrees
- moved R20 187.7 mm to (84.0, 78.1), turned to -90 degrees
- moved D8 185.7 mm to (84.0, 74.6), turned to 90 degrees
- moved J6 179.7 mm to (71.1, 77.5)
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Connections:
- TP29 pad 1: /FPGA_CDONE -> /FPGA_CRESET
- TP30 pad 1: /FPGA_CRESET -> /FPGA_CDONE
- U6 pad 14: /FPGA_CDONE -> /FPGA_CRESET
- U6 pad 15: /FPGA_CRESET -> /FPGA_CDONE
Routing:
- net +3V3: track 3.35 -> 214.9 mm, vias 0 -> 32
- net /TFT_CS: track 0.00 -> 176.0 mm
- net /TFT_SCL: track 0.00 -> 175.7 mm
- net /TFT_DCX: track 0.00 -> 175.6 mm, vias 0 -> 2
- net /TFT_SDI: track 0.00 -> 174.3 mm
- net /TFT_RESET: track 0.00 -> 154.7 mm
- net +1V2: track 0.00 -> 132.6 mm, vias 0 -> 2
- net +2V5: track 0.00 -> 119.8 mm, vias 0 -> 1
- net GND: track 0.00 -> 113.7 mm, vias 0 -> 70
- net /TFT_VSYNC: track 0.00 -> 103.0 mm, vias 0 -> 2
- net /TFT_HSYNC: track 0.00 -> 100.1 mm, vias 0 -> 2
- net /TFT_DATA_RED4: track 0.00 -> 97.5 mm
- net /TFT_DOTCLK: track 0.00 -> 96.9 mm, vias 0 -> 2
- net /TFT_DATA_RED3: track 0.00 -> 94.8 mm
- net /TFT_DE: track 0.00 -> 94.2 mm, vias 0 -> 2
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- added copper zone on In2.Cu, net +3V3
- added copper zone on In2.Cu, net +5V
- added copper zone on B.Cu, net GND
- added copper zone on In1.Cu, net GND
Other:
- board outline added: 100 x 100 mm
- copper layers 2 -> 4
